File: circuit_v3sdcard/main.sch (EAGLE design)
At the start: 29 parts, among them CN1 SD, CN2 USB_BARE, IC1 C8051F381-GM, IC3 N25Q512A, IC4 KC2016K, IC6 MPU-9250, P0.0 PTR1TP10R, SW2 PTR1TP10R

Commit message: Added connector on v3 sdcard circuit
Parts:
- added CN3: MICROSD, Connector:MICROSD
Changed lines of the file:
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@@
 <?xml version="1.0" encoding="utf-8"?>
 <!DOCTYPE eagle SYSTEM "eagle.dtd">
-<eagle version="9.0.1">
+<eagle version="9.1.3">
 <drawing>
 <settings>
@@
 <layer number="51" name="tDocu" color="7" fill="1" visible="no" active="no"/>
 <layer number="52" name="bDocu" color="7" fill="1" visible="no" active="no"/>
+<layer number="88" name="SimResults" color="9" fill="1" visible="yes" active="yes"/>
+<layer number="89" name="SimProbes" color="9" fill="1" visible="yes" active="yes"/>
+<layer number="90" name="Modules" color="5" fill="1" visible="yes" active="yes"/>
 <layer number="91" name="Nets" color="2" fill="1" visible="yes" active="yes"/>
 <layer number="92" name="Busses" color="1" fill="1" visible="yes" active="yes"/>
@@
 <part name="SUPPLY2" library="supply2" deviceset="DGND" device=""/>
 <part name="CN1" library="Connector" deviceset="SD" device=""/>
+<part name="CN3" library="Connector" deviceset="MICROSD" device=""/>
 </parts>
 <sheets>
@@
 <instance part="SUPPLY2" gate="G$1" x="-78.74" y="-17.78"/>
 <instance part="CN1" gate="G$1" x="-129.54" y="-55.88"/>
+<instance part="CN3" gate="G$1" x="-203.2" y="-58.42"/>
 </instances>
 <busses>

Commit message: Added molex connector's library
Parts:
- added CN4: 5035481020, Connector:5035481020
Changed lines of the file:
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@@
 <part name="CN1" library="Connector" deviceset="SD" device=""/>
 <part name="CN3" library="Connector" deviceset="MICROSD" device=""/>
+<part name="CN4" library="Connector" deviceset="5035481020" device=""/>
 </parts>
 <sheets>
@@
 <instance part="CN1" gate="G$1" x="-129.54" y="-55.88"/>
 <instance part="CN3" gate="G$1" x="-203.2" y="-58.42"/>
+<instance part="CN4" gate="G$1" x="-226.06" y="-45.72"/>
 </instances>
 <busses>

Commit message: Modified SD circuit
Connections:
- new net N$10: CN1.P$3, CN3.P$3
- new net N$12: CN1.P$2, CN3.P$2
- new net N$14: CN1.P$1, CN3.P$1
- new net N$2: CN1.P$9, CN3.P$8
- new net N$3: CN1.P$8, CN3.P$7
- new net N$4: CN1.P$4, CN1.P$7, CN3.P$6
- new net N$6: CN1.P$6, CN3.P$5
- new net N$8: CN1.P$5, CN3.P$4
Other:
- moved on the sheet: CN1
Changed lines of the file:
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@@
 </variantdefs>
 <classes>
-<class number="0" name="default" width="0" drill="0">
+<class number="0" name="signal" width="0.1524" drill="0">
+</class>
+<class number="1" name="power" width="0.254" drill="0">
 </class>
 </classes>
@@
 <instance part="R1" gate="G$1" x="-78.74" y="-12.7" rot="R90"/>
 <instance part="SUPPLY2" gate="G$1" x="-78.74" y="-17.78"/>
-<instance part="CN1" gate="G$1" x="-129.54" y="-55.88"/>
+<instance part="CN1" gate="G$1" x="-172.72" y="-55.88" rot="MR0"/>
 <instance part="CN3" gate="G$1" x="-203.2" y="-58.42"/>
 <instance part="CN4" gate="G$1" x="-226.06" y="-45.72"/>
@@
 </segment>
 </net>
+<net name="N$2" class="0">
+<segment>
+<pinref part="CN3" gate="G$1" pin="P$8"/>
+<pinref part="CN1" gate="G$1" pin="P$9"/>
+<wire x1="-198.12" y1="-66.04" x2="-175.26" y2="-66.04" width="0.1524" layer="91"/>
+</segment>
+</net>
+<net name="N$3" class="0">
+<segment>
+<pinref part="CN1" gate="G$1" pin="P$8"/>
+<pinref part="CN3" gate="G$1" pin="P$7"/>
+<wire x1="-175.26" y1="-63.5" x2="-198.12" y2="-63.5" width="0.1524" layer="91"/>
+</segment>
+</net>
+<net name="N$4" class="0">
+<segment>
+<pinref part="CN3" gate="G$1" pin="P$6"/>
+<pinref part="CN1" gate="G$1" pin="P$7"/>
+<wire x1="-198.12" y1="-60.96" x2="-185.42" y2="-60.96" width="0.1524" layer="91"/>
+<pinref part="CN1" gate="G$1" pin="P$4"/>
+<wire x1="-185.42" y1="-60.96" x2="-175.26" y2="-60.96" width="0.1524" layer="91"/>
+<wire x1="-175.26" y1="-53.34" x2="-185.42" y2="-53.34" width="0.1524" layer="91"/>
+<wire x1="-185.42" y1="-53.34" x2="-185.42" y2="-60.96" width="0.1524" layer="91"/>
+<junction x="-185.42" y="-60.96"/>
+</segment>
+</net>
+<net name="N$6" class="0">
+<segment>
+<pinref part="CN1" gate="G$1" pin="P$6"/>
+<pinref part="CN3" gate="G$1" pin="P$5"/>
+<wire x1="-175.26" y1="-58.42" x2="-198.12" y2="-58.42" width="0.1524" layer="91"/>
+</segment>
+</net>
+<net name="N$8" class="0">
+<segment>
+<pinref part="CN3" gate="G$1" pin="P$4"/>
+<pinref part="CN1" gate="G$1" pin="P$5"/>
+<wire x1="-198.12" y1="-55.88" x2="-175.26" y2="-55.88" width="0.1524" layer="91"/>
+</segment>
+</net>
+<net name="N$10" class="0">
+<segment>
+<pinref part="CN1" gate="G$1" pin="P$3"/>
+<wire x1="-175.26" y1="-50.8" x2="-187.96" y2="-50.8" width="0.1524" layer="91"/>
+<wire x1="-187.96" y1="-50.8" x2="-187.96" y2="-53.34" width="0.1524" layer="91"/>
+<pinref part="CN3" gate="G$1" pin="P$3"/>
+<wire x1="-187.96" y1="-53.34" x2="-198.12" y2="-53.34" width="0.1524" layer="91"/>
+</segment>
+</net>
+<net name="N$12" class="0">
+<segment>
+<pinref part="CN1" gate="G$1" pin="P$2"/>
+<wire x1="-175.26" y1="-48.26" x2="-190.5" y2="-48.26" width="0.1524" layer="91"/>
+<wire x1="-190.5" y1="-48.26" x2="-190.5" y2="-50.8" width="0.1524" layer="91"/>
+<pinref part="CN3" gate="G$1" pin="P$2"/>
+<wire x1="-190.5" y1="-50.8" x2="-198.12" y2="-50.8" width="0.1524" layer="91"/>
+</segment>
+</net>
+<net name="N$14" class="0">
+<segment>
+<pinref part="CN3" gate="G$1" pin="P$1"/>
+<wire x1="-198.12" y1="-48.26" x2="-193.04" y2="-48.26" width="0.1524" layer="91"/>
+<wire x1="-193.04" y1="-48.26" x2="-193.04" y2="-45.72" width="0.1524" layer="91"/>
+<pinref part="CN1" gate="G$1" pin="P$1"/>
+<wire x1="-193.04" y1="-45.72" x2="-175.26" y2="-45.72" width="0.1524" layer="91"/>
+</segment>
+</net>
